Commit message: Rename tip_link to tcp_link

File: aist_robotiq/urdf/robotiq_140_gripper.urdf.xacro (robot description, xacro)
@@ -252,7 +252,7 @@
       <origin xyz="0 0 0" rpy="${pi} ${-pi/2} 0"/>
     </joint>
-    <joint name="${prefix}tip_link_joint" type="fixed">
+    <joint name="${prefix}tcp_link_joint" type="fixed">
       <parent link="${prefix}base_link"/>
-      <child link="${prefix}tip_link"/>
+      <child link="${prefix}tcp_link"/>
       <xacro:if value="${short_finger}">
 	<origin rpy="0.0 ${-pi/2} 0.0" xyz=".2053 0.0 0.0"/>
@@ -262,5 +262,5 @@
       </xacro:unless>
     </joint>
-    <link name="${prefix}tip_link"/>
+    <link name="${prefix}tcp_link"/>
     <xacro:robotiq_arg2f_base_link prefix="${prefix}"/>
     <xacro:finger_links prefix="${prefix}" fingerprefix="left"

File: aist_robotiq/urdf/robotiq_3f_gripper.urdf.xacro (robot description, xacro)
@@ -3,5 +3,5 @@
        xmlns:xacro="http://ros.org/wiki/xacro">
   <xacro:macro name="robotiq_3f_gripper" params="prefix parent *origin">
-    <xacro:property name="tip_height"		value="0.204"/>
+    <xacro:property name="tcp_height"		value="0.204"/>
     <xacro:property name="distal_length"	value="0.0335"/>
     <xacro:property name="distal_offset"	value="0.0095"/>
@@ -182,7 +182,7 @@
     </link>
     <!-- Gripper tip -->
-    <xacro:set_frame name="${prefix}tip_link"
+    <xacro:set_frame name="${prefix}tcp_link"
 		     parent="${prefix}base_link">
-      <origin xyz="${tip_height} 0.0 0.0" rpy="0 ${radians(-90)} 0"/>
+      <origin xyz="${tcp_height} 0.0 0.0" rpy="0 ${radians(-90)} 0"/>
     </xacro:set_frame>
     <!-- middle finger -->

File: aist_robotiq/urdf/robotiq_85_gripper.urdf.xacro (robot description, xacro)
@@ -235,10 +235,10 @@
       <origin xyz="0 0 0" rpy="${pi} ${-pi/2} 0"/>
     </joint>
-    <joint name="${prefix}tip_link_joint" type="fixed">
+    <joint name="${prefix}tcp_link_joint" type="fixed">
       <parent link="${prefix}base_link"/>
-      <child link="${prefix}tip_link"/>
+      <child link="${prefix}tcp_link"/>
       <origin rpy="0.0 ${-pi/2} 0.0" xyz="0.1628 0.0 0.0"/>
     </joint>
-    <link name="${prefix}tip_link"/>
+    <link name="${prefix}tcp_link"/>
     <xacro:robotiq_arg2f_base_link prefix="${prefix}"/>
     <xacro:finger_links prefix="${prefix}" fingerprefix="left" stroke="85"/>

File: aist_robotiq/urdf/robotiq_epick_gripper.urdf.xacro (robot description, xacro)
@@ -76,8 +76,8 @@
 	<origin xyz="0 0 0" rpy="0 0 0"/>
       </joint>
-      <link name="${prefix}tip_link"/>
+      <link name="${prefix}tcp_link"/>
       <joint name="${prefix}tip_joint" type="fixed">
 	<parent link="${prefix}plunger_link"/>
-	<child  link="${prefix}tip_link"/>
+	<child  link="${prefix}tcp_link"/>
 	<origin xyz="${plunger_length} 0 0" rpy="0 ${-pi/2} 0"/>
       </joint>

File: aist_robotiq/urdf/robotiq_hande_gripper.urdf.xacro (robot description, xacro)
@@ -19,10 +19,10 @@
       <origin xyz="0 0 0" rpy="${pi/2} 0 ${pi/2}"/>
     </joint>
-    <joint name="${prefix}tip_link_joint" type="fixed">
+    <joint name="${prefix}tcp_link_joint" type="fixed">
       <parent link="${prefix}base_link"/>
-      <child link="${prefix}tip_link"/>
+      <child link="${prefix}tcp_link"/>
       <origin rpy="0.0 ${-pi/2} 0.0" xyz=".146 0.0 0.0"/>
     </joint>
-    <link name="${prefix}tip_link"/>
+    <link name="${prefix}tcp_link"/>
     <link name="${prefix}hande_link">
       <inertial>

Commit message: Revert "Rename tip_link to tcp_link"
This reverts commit f2397edaf7b29da5a105f061aa89e3820c892c00.

File: aist_robotiq/urdf/robotiq_140_gripper.urdf.xacro (robot description, xacro)
@@ -252,7 +252,7 @@
       <origin xyz="0 0 0" rpy="${pi} ${-pi/2} 0"/>
     </joint>
-    <joint name="${prefix}tcp_link_joint" type="fixed">
+    <joint name="${prefix}tip_link_joint" type="fixed">
       <parent link="${prefix}base_link"/>
-      <child link="${prefix}tcp_link"/>
+      <child link="${prefix}tip_link"/>
       <xacro:if value="${short_finger}">
 	<origin rpy="0.0 ${-pi/2} 0.0" xyz=".2053 0.0 0.0"/>
@@ -262,5 +262,5 @@
       </xacro:unless>
     </joint>
-    <link name="${prefix}tcp_link"/>
+    <link name="${prefix}tip_link"/>
     <xacro:robotiq_arg2f_base_link prefix="${prefix}"/>
     <xacro:finger_links prefix="${prefix}" fingerprefix="left"

File: aist_robotiq/urdf/robotiq_3f_gripper.urdf.xacro (robot description, xacro)
@@ -3,5 +3,5 @@
        xmlns:xacro="http://ros.org/wiki/xacro">
   <xacro:macro name="robotiq_3f_gripper" params="prefix parent *origin">
-    <xacro:property name="tcp_height"		value="0.204"/>
+    <xacro:property name="tip_height"		value="0.204"/>
     <xacro:property name="distal_length"	value="0.0335"/>
     <xacro:property name="distal_offset"	value="0.0095"/>
@@ -182,7 +182,7 @@
     </link>
     <!-- Gripper tip -->
-    <xacro:set_frame name="${prefix}tcp_link"
+    <xacro:set_frame name="${prefix}tip_link"
 		     parent="${prefix}base_link">
-      <origin xyz="${tcp_height} 0.0 0.0" rpy="0 ${radians(-90)} 0"/>
+      <origin xyz="${tip_height} 0.0 0.0" rpy="0 ${radians(-90)} 0"/>
     </xacro:set_frame>
     <!-- middle finger -->

File: aist_robotiq/urdf/robotiq_85_gripper.urdf.xacro (robot description, xacro)
@@ -235,10 +235,10 @@
       <origin xyz="0 0 0" rpy="${pi} ${-pi/2} 0"/>
     </joint>
-    <joint name="${prefix}tcp_link_joint" type="fixed">
+    <joint name="${prefix}tip_link_joint" type="fixed">
       <parent link="${prefix}base_link"/>
-      <child link="${prefix}tcp_link"/>
+      <child link="${prefix}tip_link"/>
       <origin rpy="0.0 ${-pi/2} 0.0" xyz="0.1628 0.0 0.0"/>
     </joint>
-    <link name="${prefix}tcp_link"/>
+    <link name="${prefix}tip_link"/>
     <xacro:robotiq_arg2f_base_link prefix="${prefix}"/>
     <xacro:finger_links prefix="${prefix}" fingerprefix="left" stroke="85"/>

File: aist_robotiq/urdf/robotiq_epick_gripper.urdf.xacro (robot description, xacro)
@@ -76,8 +76,8 @@
 	<origin xyz="0 0 0" rpy="0 0 0"/>
       </joint>
-      <link name="${prefix}tcp_link"/>
+      <link name="${prefix}tip_link"/>
       <joint name="${prefix}tip_joint" type="fixed">
 	<parent link="${prefix}plunger_link"/>
-	<child  link="${prefix}tcp_link"/>
+	<child  link="${prefix}tip_link"/>
 	<origin xyz="${plunger_length} 0 0" rpy="0 ${-pi/2} 0"/>
       </joint>

File: aist_robotiq/urdf/robotiq_hande_gripper.urdf.xacro (robot description, xacro)
@@ -19,10 +19,10 @@
       <origin xyz="0 0 0" rpy="${pi/2} 0 ${pi/2}"/>
     </joint>
-    <joint name="${prefix}tcp_link_joint" type="fixed">
+    <joint name="${prefix}tip_link_joint" type="fixed">
       <parent link="${prefix}base_link"/>
-      <child link="${prefix}tcp_link"/>
+      <child link="${prefix}tip_link"/>
       <origin rpy="0.0 ${-pi/2} 0.0" xyz=".146 0.0 0.0"/>
     </joint>
-    <link name="${prefix}tcp_link"/>
+    <link name="${prefix}tip_link"/>
     <link name="${prefix}hande_link">
       <inertial>
